Commit message: Smartdumpster simulation base

File: smartdumpster2_ws/src/smartdumpster_description/urdf/sdumpster.urdf.xacro (robot description, xacro)
@@ -1,6 +1,14 @@
 <?xml version="1.0"?>
 <robot xmlns:xacro="http://www.ros.org/wiki/xacro" name="smartdumpster">
+    <xacro:include filename="$(find smartdumpster_description)/urdf/sdumpster_gazebo.xacro" />
     <link name="base_footprint" />
     <link name="base_link">
+        <inertial>
+            <mass value="40.0" />
+            <origin xyz="0 0 0" rpy="0 0 0" />
+            <inertia ixx="3.27" ixy="0.0" ixz="0.0"
+                     iyy="3.77" iyz="0.0"
+                     izz="3.77" />
+        </inertial>
         <visual>
             <origin rpy="1.57 0 1.57" xyz="0 0 0" />
@@ -9,11 +17,24 @@
             </geometry>
         </visual>
+        <collision>
+            <origin rpy="1.57 0 1.57" xyz="0 0 0" />
+            <geometry>
+                <mesh filename="package://smartdumpster_description/meshes/base_link.stl" scale="0.001 0.001 0.001" />
+            </geometry>
+        </collision>
     </link>
     <joint name="base_joint" type="fixed">
         <parent link="base_footprint" />
         <child link="base_link" />
-        <origin rpy="0 0 0" xyz="0 0 0.0995" />
+        <origin rpy="0 0 0" xyz="0 0 0.1175" />
     </joint>
     <link name="wheel_right_link">
+        <inertial>
+            <mass value="0.836" />
+            <origin xyz="0 0 0" rpy="0 0 0" />
+            <inertia ixx="0.00397" ixy="0.0" ixz="0.0"
+                     iyy="0.00210" iyz="0.0"
+                     izz="0.00210" />
+        </inertial>
         <visual>
             <origin rpy="0 0 1.57" xyz="0 0 0" />
@@ -22,4 +43,10 @@
             </geometry>
         </visual>
+        <collision>
+            <origin rpy="0 0 1.57" xyz="0 -0.015 0" />
+            <geometry>
+                <sphere radius="0.0975" />
+            </geometry>
+        </collision>
     </link>
     <joint name="wheel_right_joint" type="continuous">
@@ -30,4 +57,11 @@
     </joint>
     <link name="wheel_left_link">
+        <inertial>
+            <mass value="0.836" />
+            <origin xyz="0 0 0" rpy="0 0 0" />
+            <inertia ixx="0.00397" ixy="0.0" ixz="0.0"
+                     iyy="0.00210" iyz="0.0"
+                     izz="0.00210" />
+        </inertial>
         <visual>
             <origin rpy="0 0 1.57" xyz="0 0 0" />
@@ -36,4 +70,10 @@
             </geometry>
         </visual>
+        <collision>
+            <origin rpy="0 0 1.57" xyz="0 0.015 0" />
+            <geometry>
+                <sphere radius="0.0975" />
+            </geometry>
+        </collision>
     </link>
     <joint name="wheel_left_joint" type="continuous">
@@ -44,4 +84,11 @@
     </joint>
     <link name="caster_front_link">
+        <inertial>
+            <mass value="0.329" />
+            <origin xyz="0 0 0" rpy="0 0 0" />
+            <inertia ixx="0.000306" ixy="0.0" ixz="0.0"
+                     iyy="0.000306" iyz="0.0"
+                     izz="0.000306" />
+        </inertial>
         <visual>
             <origin rpy="1.57 0 0" xyz="0 0 0" />
@@ -50,4 +97,10 @@
             </geometry>
         </visual>
+        <collision>
+            <origin rpy="1.57 0 0" xyz="0 0 0" />
+            <geometry>
+                <sphere radius="0.0965" />
+            </geometry>
+        </collision>
     </link>
     <joint name="caster_front_joint" type="fixed">
@@ -57,4 +110,11 @@
     </joint>
     <link name="caster_rear_link">
+        <inertial>
+            <mass value="0.329" />
+            <origin xyz="0 0 0" rpy="0 0 0" />
+            <inertia ixx="0.000306" ixy="0.0" ixz="0.0"
+                     iyy="0.000306" iyz="0.0"
+                     izz="0.000306" />
+        </inertial>
         <visual>
             <origin rpy="1.57 0 0" xyz="0 0 0" />
@@ -63,4 +123,10 @@
             </geometry>
         </visual>
+        <collision>
+            <origin rpy="1.57 0 0" xyz="0 0 0" />
+            <geometry>
+                <sphere radius="0.0965" />
+            </geometry>
+        </collision>
     </link>
     <joint name="caster_rear_joint" type="fixed">

Commit message: Kalman filter

File: smartdumpster2_ws/src/smartdumpster_description/urdf/sdumpster.urdf.xacro (robot description, xacro)
@@ -139,3 +139,30 @@
         <origin rpy="0 0 0" xyz="-0.275 0 -0.021" />
     </joint>
+    <link name="imu_link">
+        <inertial>
+            <origin xyz="-0.00552433659106688 0.000168210391520346 0.000514000497342681" rpy="0 0 0" />
+            <mass value="0.000528415362211671" />
+            <inertia ixx="1.46176048428261E-08" ixy="1.40015117949421E-10" ixz="-1.99633872937403E-12"
+                    iyy="8.59662482954888E-09" iyz="7.52375112767959E-12"
+                    izz="2.30279421279312E-08" />
+        </inertial>
+        <visual>
+            <origin rpy="0 0 0" xyz="0 0 0" />
+            <geometry>
+                <mesh filename="package://smartdumpster_description/meshes/imu_link.STL" />
+            </geometry>
+        </visual>
+        <collision>
+            <origin rpy="0 0 0" xyz="0 0 0" />
+            <geometry>
+                <mesh filename="package://smartdumpster_description/meshes/imu_link.STL" />
+            </geometry>
+        </collision>
+    </link>
+    <joint name="imu_joint" type="fixed">
+        <parent link="base_link" />
+        <child link="imu_link" />
+        <axis xyz="0 0 0" />
+        <origin xyz="0 0 0.150" rpy="0 0 0" />
+    </joint>
 </robot>

File: smartdumpster2_ws/src/smartdumpster_description/urdf/sdumpster_gazebo.xacro (robot description, xacro)
@@ -35,8 +35,11 @@
         <maxVel>0.1</maxVel>
     </gazebo>
+    <!-- ROS 2 Control -->
     <gazebo>
         <xacro:if value="$(arg is_ignition)">
             <plugin filename="ign_ros2_control-system" name="ign_ros2_control::IgnitionROS2ControlPlugin">
                 <parameters>$(find smartdumpster_controller)/config/sdumpster_controllers.yaml</parameters>
+            </plugin>
+            <plugin filename="ignition-gazebo-imu-system" name="ignition::gazebo::systems::Imu">
             </plugin>
         </xacro:if>
@@ -45,5 +48,57 @@
                 <parameters>$(find smartdumpster_controller)/config/sdumpster_controllers.yaml</parameters>
             </plugin>
+            <plugin filename="gz-sim-imu-system" name="gz::sim::systems::Imu">
+            </plugin>
         </xacro:unless>
     </gazebo>
+    <gazebo reference="imu_link">
+        <sensor name="imu" type="imu">
+            <always_on>true</always_on>
+            <update_rate>100</update_rate>
+            <gz_frame_id>imu_link</gz_frame_id>
+            <topic>imu</topic>
+            <imu>
+                <angular_velocity>
+                    <x>
+                        <noise type="gaussian">
+                            <mean>0.0</mean>
+                            <stddev>2e-4</stddev>
+                        </noise>
+                    </x>
+                    <y>
+                        <noise type="gaussian">
+                            <mean>0.0</mean>
+                            <stddev>2e-4</stddev>
+                        </noise>
+                    </y>
+                    <z>
+                        <noise type="gaussian">
+                            <mean>0.0</mean>
+                            <stddev>2e-4</stddev>
+                        </noise>
+                    </z>
+                </angular_velocity>
+                <linear_acceleration>
+                    <x>
+                        <noise type="gaussian">
+                            <mean>0.0</mean>
+                            <stddev>1.7e-2</stddev>
+                        </noise>
+                    </x>
+                    <y>
+                        <noise type="gaussian">
+                            <mean>0.0</mean>
+                            <stddev>1.7e-2</stddev>
+                        </noise>
+                    </y>
+                    <z>
+                        <noise type="gaussian">
+                            <mean>0.0</mean>
+                            <stddev>1.7e-2</stddev>
+                        </noise>
+                    </z>
+                </linear_acceleration>
+            </imu>
+        </sensor>
+    </gazebo>
 </robot>

Commit message: Laser 2D simulation & virtual enviorment

File: smartdumpster2_ws/src/smartdumpster_description/urdf/sdumpster.urdf.xacro (robot description, xacro)
@@ -21,4 +21,5 @@
                 <mesh filename="package://smartdumpster_description/meshes/base_link.stl" scale="0.001 0.001 0.001" />
             </geometry>
+            <material name="silver"/>
         </visual>
         <collision>
@@ -47,4 +48,5 @@
                 <mesh filename="package://smartdumpster_description/meshes/wheel_right_link.stl" scale="0.001 0.001 0.001" />
             </geometry>
+            <material name="black"/>
         </visual>
         <collision>
@@ -74,4 +76,5 @@
                 <mesh filename="package://smartdumpster_description/meshes/wheel_left_link.stl" scale="0.001 0.001 0.001" />
             </geometry>
+            <material name="black"/>
         </visual>
         <collision>
@@ -101,4 +104,5 @@
                 <mesh filename="package://smartdumpster_description/meshes/caster_wheel_link.stl" scale="0.001 0.001 0.001" />
             </geometry>
+            <material name="black"/>
         </visual>
         <collision>
@@ -127,4 +131,5 @@
                 <mesh filename="package://smartdumpster_description/meshes/caster_wheel_link.stl" scale="0.001 0.001 0.001" />
             </geometry>
+            <material name="black"/>
         </visual>
         <collision>
@@ -167,3 +172,44 @@
         <origin xyz="0 0 0.150" rpy="0 0 0" />
     </joint>
+    <link name="laser_link">
+        <inertial>
+            <origin xyz="-0.011945780406062 -0.000381929217680526 -0.0170649378129477" rpy="0 0 0" />
+            <mass value="0.073084435549317" />
+            <inertia ixx="1.96074931730795E-05" ixy="-3.62091076640009E-07" ixz="4.28230084046735E-07"
+                     iyy="2.40983835136327E-05" iyz="1.50180909250652E-08"
+                     izz="4.14184164228595E-05" />
+        </inertial>
+        <visual>
+            <origin rpy="0 0 0" xyz="0 0 0" />
+            <geometry>
+                <mesh filename="package://smartdumpster_description/meshes/laser_link.STL" />
+            </geometry>
+            <material name="dark_grey"/>
+        </visual>
+        <collision>
+            <origin rpy="0 0 0" xyz="0 0 0" />
+            <geometry>
+                <mesh filename="package://smartdumpster_description/meshes/laser_link.STL" />
+            </geometry>
+        </collision>
+    </link>
+    <joint name="laser_joint" type="fixed">
+        <parent link="base_link" />
+        <child link="laser_link" />
+        <axis xyz="0 0 0" />
+        <origin xyz="0 0 0.1808" rpy="0 0 3.14" />
+    </joint>
+    <!-- VISUAL MATERIAL COLOR -->
+    <material name="blue">
+        <color rgba="0 0 1 1"/>
+    </material>
+    <material name="black">
+        <color rgba="0 0 0 1"/>
+    </material>
+    <material name="silver">
+        <color rgba="0.79 0.82 0.93 1"/>
+    </material>
+    <material name="dark_grey">
+        <color rgba="0.3 0.3 0.3 1"/>
+    </material>
 </robot>

File: smartdumpster2_ws/src/smartdumpster_description/urdf/sdumpster_gazebo.xacro (robot description, xacro)
@@ -43,4 +43,7 @@
             <plugin filename="ignition-gazebo-imu-system" name="ignition::gazebo::systems::Imu">
             </plugin>
+            <plugin filename="ignition-gazebo-sensors-system" name="ignition::gazebo::systems::Sensors">
+                <render_engine>ogre2</render_engine>
+            </plugin>
         </xacro:if>
         <xacro:unless value="$(arg is_ignition)">
@@ -50,6 +53,10 @@
             <plugin filename="gz-sim-imu-system" name="gz::sim::systems::Imu">
             </plugin>
+            <plugin filename="gz-sim-sensors-system" name="gz::sim::systems::Sensors">
+                <render_engine>ogre2</render_engine>
+            </plugin>
         </xacro:unless>
     </gazebo>
+    <!-- IMU Sensor -->
     <gazebo reference="imu_link">
         <sensor name="imu" type="imu">
@@ -102,3 +109,33 @@
         </sensor>
     </gazebo>
+    <!-- LIDAR Sensor -->
+    <gazebo reference="laser_link">
+        <sensor name="lidar" type="gpu_ray">
+            <always_on>true</always_on>
+            <visualize>true</visualize>
+            <topic>scan</topic>
+            <update_rate>5</update_rate>
+            <gz_frame_id>laser_link</gz_frame_id>
+            <lidar>
+                <scan>
+                <horizontal>
+                    <samples>360</samples>
+                    <resolution>1.00000</resolution>
+                    <min_angle>0.000000</min_angle>
+                    <max_angle>6.280000</max_angle>
+                </horizontal>
+                </scan>
+                <range>
+                <min>0.120000</min>
+                <max>12.0</max>
+                <resolution>0.02</resolution>
+                </range>
+                <noise>
+                <type>gaussian</type>
+                <mean>0.0</mean>
+                <stddev>0.01</stddev>
+                </noise>
+            </lidar>
+        </sensor>
+    </gazebo>
 </robot>

Commit message: New localization + Zed2i simulation implementation

File: smartdumpster2_ws/src/smartdumpster_description/urdf/sdumpster.urdf.xacro (robot description, xacro)
@@ -145,4 +145,43 @@
         <origin rpy="0 0 0" xyz="-0.275 0 -0.021" />
     </joint>
+    <!-- Laser 2D -->
+    <link name="laser_link">
+        <inertial>
+            <origin xyz="-0.011945780406062 -0.000381929217680526 -0.0170649378129477" rpy="0 0 0" />
+            <mass value="0.073084435549317" />
+            <inertia ixx="1.96074931730795E-05" ixy="-3.62091076640009E-07" ixz="4.28230084046735E-07"
+                     iyy="2.40983835136327E-05" iyz="1.50180909250652E-08"
+                     izz="4.14184164228595E-05" />
+        </inertial>
+        <visual>
+            <origin rpy="0 0 0" xyz="0 0 0" />
+            <geometry>
+                <mesh filename="package://smartdumpster_description/meshes/laser_link.STL" />
+            </geometry>
+            <material name="dark_grey"/>
+        </visual>
+        <collision>
+            <origin rpy="0 0 0" xyz="0 0 0" />
+            <geometry>
+                <mesh filename="package://smartdumpster_description/meshes/laser_link.STL" />
+            </geometry>
+        </collision>
+    </link>
+    <joint name="laser_joint" type="fixed">
+        <parent link="base_link" />
+        <child link="laser_link" />
+        <axis xyz="0 0 0" />
+        <origin xyz="0 0 0.1808" rpy="0 0 3.14" />
+    </joint>
+    <!-- Zed2i Camera + Sensor Integrated -->
+    <xacro:include filename="$(find zed_description)/urdf/zed_macro.urdf.xacro" />
+    <xacro:zed_camera name="zed2i" model="zed2i" enable_gnss="false">
+        <origin xyz="0 0 0" rpy="0 0 0" />
+    </xacro:zed_camera>
+    <joint name="zed2i_base_joint" type="fixed">
+        <parent link="base_link" />
+        <child link="zed2i_camera_link" />
+        <origin xyz="0.399 0 0.075" rpy="0 0 0" />
+    </joint>
     <link name="imu_link">
         <inertial>
@@ -167,36 +206,8 @@
     </link>
     <joint name="imu_joint" type="fixed">
-        <parent link="base_link" />
+        <parent link="zed2i_left_camera_frame" />
         <child link="imu_link" />
         <axis xyz="0 0 0" />
-        <origin xyz="0 0 0.150" rpy="0 0 0" />
-    </joint>
-    <link name="laser_link">
-        <inertial>
-            <origin xyz="-0.011945780406062 -0.000381929217680526 -0.0170649378129477" rpy="0 0 0" />
-            <mass value="0.073084435549317" />
-            <inertia ixx="1.96074931730795E-05" ixy="-3.62091076640009E-07" ixz="4.28230084046735E-07"
-                     iyy="2.40983835136327E-05" iyz="1.50180909250652E-08"
-                     izz="4.14184164228595E-05" />
-        </inertial>
-        <visual>
-            <origin rpy="0 0 0" xyz="0 0 0" />
-            <geometry>
-                <mesh filename="package://smartdumpster_description/meshes/laser_link.STL" />
-            </geometry>
-            <material name="dark_grey"/>
-        </visual>
-        <collision>
-            <origin rpy="0 0 0" xyz="0 0 0" />
-            <geometry>
-                <mesh filename="package://smartdumpster_description/meshes/laser_link.STL" />
-            </geometry>
-        </collision>
-    </link>
-    <joint name="laser_joint" type="fixed">
-        <parent link="base_link" />
-        <child link="laser_link" />
-        <axis xyz="0 0 0" />
-        <origin xyz="0 0 0.1808" rpy="0 0 3.14" />
+        <origin xyz="-0.002 -0.023 0.00022" rpy="-0.004 0.00 -0.008" />
     </joint>
     <!-- VISUAL MATERIAL COLOR -->

File: smartdumpster2_ws/src/smartdumpster_description/urdf/sdumpster_gazebo.xacro (robot description, xacro)
@@ -58,11 +58,61 @@
         </xacro:unless>
     </gazebo>
-    <!-- IMU Sensor -->
+    <!-- LIDAR Sensor -->
+    <gazebo reference="laser_link">
+        <sensor name="lidar" type="gpu_ray">
+            <always_on>true</always_on>
+            <visualize>true</visualize>
+            <topic>scan</topic>
+            <update_rate>5</update_rate>
+            <gz_frame_id>laser_link</gz_frame_id>
+            <lidar>
+                <scan>
+                <horizontal>
+                    <samples>360</samples>
+                    <resolution>1.00000</resolution>
+                    <min_angle>0.000000</min_angle>
+                    <max_angle>6.280000</max_angle>
+                </horizontal>
+                </scan>
+                <range>
+                <min>0.120000</min>
+                <max>12.0</max>
+                <resolution>0.02</resolution>
+                </range>
+                <noise>
+                <type>gaussian</type>
+                <mean>0.0</mean>
+                <stddev>0.01</stddev>
+                </noise>
+            </lidar>
+        </sensor>
+    </gazebo>
+    <!-- Zed2i Camera -->
+    <gazebo reference="zed2i_camera_link">
+        <sensor name="zed2i_rgbd" type="rgbd_camera">
+            <pose>0 0 0 0 0 0</pose>
+            <camera>
+                <horizontal_fov>1.92</horizontal_fov>
+                <image>
+                    <width>640</width>
+                    <height>480</height>
+                </image>
+                <clip>
+                    <near>0.1</near>
+                    <far>100</far>
+                </clip>
+                <optical_frame_id>zed2i_camera_center</optical_frame_id>
+            </camera>
+            <always_on>1</always_on>
+            <update_rate>10</update_rate>
+            <visualize>true</visualize>
+            <topic>zed2i</topic>
+            <frame_id>zed2i_camera_link</frame_id>
+            <gz_frame_id>zed2i_camera_link</gz_frame_id>
+        </sensor>
+    </gazebo>
     <gazebo reference="imu_link">
+        <!-- IMU Sensor -->
         <sensor name="imu" type="imu">
-            <always_on>true</always_on>
-            <update_rate>100</update_rate>
-            <gz_frame_id>imu_link</gz_frame_id>
-            <topic>imu</topic>
             <imu>
                 <angular_velocity>
@@ -107,34 +157,8 @@
                 </linear_acceleration>
             </imu>
-        </sensor>
-    </gazebo>
-    <!-- LIDAR Sensor -->
-    <gazebo reference="laser_link">
-        <sensor name="lidar" type="gpu_ray">
             <always_on>true</always_on>
-            <visualize>true</visualize>
-            <topic>scan</topic>
-            <update_rate>5</update_rate>
-            <gz_frame_id>laser_link</gz_frame_id>
-            <lidar>
-                <scan>
-                <horizontal>
-                    <samples>360</samples>
-                    <resolution>1.00000</resolution>
-                    <min_angle>0.000000</min_angle>
-                    <max_angle>6.280000</max_angle>
-                </horizontal>
-                </scan>
-                <range>
-                <min>0.120000</min>
-                <max>12.0</max>
-                <resolution>0.02</resolution>
-                </range>
-                <noise>
-                <type>gaussian</type>
-                <mean>0.0</mean>
-                <stddev>0.01</stddev>
-                </noise>
-            </lidar>
+            <update_rate>100</update_rate>
+            <gz_frame_id>zed2i_camera_link</gz_frame_id>
+            <topic>zed2i/imu</topic>
         </sensor>
     </gazebo>
