Commit message: Remote commit

File: smartdumpster2_ws/src/smartdumpster_description/urdf/sdumpster.urdf.xacro (robot description, xacro)
@@ -145,32 +145,32 @@
         <origin rpy="0 0 0" xyz="-0.275 0 -0.021" />
     </joint>
-    <!-- Laser 2D -->
-    <link name="laser_link">
-        <inertial>
-            <origin xyz="-0.011945780406062 -0.000381929217680526 -0.0170649378129477" rpy="0 0 0" />
-            <mass value="0.073084435549317" />
-            <inertia ixx="1.96074931730795E-05" ixy="-3.62091076640009E-07" ixz="4.28230084046735E-07"
-                     iyy="2.40983835136327E-05" iyz="1.50180909250652E-08"
-                     izz="4.14184164228595E-05" />
-        </inertial>
-        <visual>
-            <origin rpy="0 0 0" xyz="0 0 0" />
-            <geometry>
-                <mesh filename="package://smartdumpster_description/meshes/laser_link.STL" />
-            </geometry>
-            <material name="dark_grey"/>
-        </visual>
-        <collision>
-            <origin rpy="0 0 0" xyz="0 0 0" />
-            <geometry>
-                <mesh filename="package://smartdumpster_description/meshes/laser_link.STL" />
-            </geometry>
-        </collision>
-    </link>
-    <joint name="laser_joint" type="fixed">
-        <parent link="base_link" />
-        <child link="laser_link" />
+    <!-- GPS RTK -->
+    <link name="gps_link">
+        <inertial>
+            <origin xyz="0 0 0" rpy="0 0 0" />
+            <mass value="0.1" />
+            <inertia ixx="0.0001" ixy="0.0" ixz="0.0"
+                     iyy="0.0001" iyz="0.0"
+                     izz="0.0002" />
+        </inertial>
+        <visual>
+            <origin rpy="1.57 0 0" xyz="0 0 0" />
+            <geometry>
+                <mesh filename="package://smartdumpster_description/meshes/gps_link.stl" scale="0.001 0.001 0.001" />
+            </geometry>
+            <material name="blue"/>
+        </visual>
+        <collision>
+            <origin rpy="1.57 0 0" xyz="0 0 0" />
+            <geometry>
+                <cylinder radius="0.06" length="0.02"/>
+            </geometry>
+        </collision>
+    </link>
+    <joint name="gps_joint" type="fixed">
+        <parent link="base_link" />
+        <child link="gps_link" />
         <axis xyz="0 0 0" />
-        <origin xyz="0 0 0.1808" rpy="0 0 3.14" />
+        <origin xyz="0 0 0.150" rpy="0 0 0" />
     </joint>
     <!-- Zed2i Camera + Sensor Integrated -->
@@ -182,5 +182,5 @@
         <parent link="base_link" />
         <child link="zed2i_camera_link" />
-        <origin xyz="0.399 0 0.075" rpy="0 0 0" />
+        <origin xyz="0.400 0 0.075" rpy="0 0 0" />
     </joint>
     <link name="imu_link">

File: smartdumpster2_ws/src/smartdumpster_description/urdf/sdumpster_gazebo.xacro (robot description, xacro)
@@ -53,4 +53,12 @@
             <plugin filename="gz-sim-imu-system" name="gz::sim::systems::Imu">
             </plugin>
+            <plugin filename="gz-sim-navsat-system" name="gz::sim::systems::NavSat">
+            </plugin>
+            <plugin filename="gz-sim-odometry-publisher-system" name="gz::sim::systems::OdometryPublisher">
+                <odom_topic>/ground_truth/odometry</odom_topic>
+                <odom_frame>map</odom_frame>
+                <robot_base_frame>base_footprint</robot_base_frame>
+                <publish_odom_to_tf>false</publish_odom_to_tf>
+            </plugin>
             <plugin filename="gz-sim-sensors-system" name="gz::sim::systems::Sensors">
                 <render_engine>ogre2</render_engine>
@@ -58,32 +66,27 @@
         </xacro:unless>
     </gazebo>
-    <!-- LIDAR Sensor -->
-    <gazebo reference="laser_link">
-        <sensor name="lidar" type="gpu_ray">
+    <!-- GPS RTK -->
+    <gazebo reference="gps_link">
+        <sensor name="gps_rtk" type="navsat">
             <always_on>true</always_on>
-            <visualize>true</visualize>
-            <topic>scan</topic>
-            <update_rate>5</update_rate>
-            <gz_frame_id>laser_link</gz_frame_id>
-            <lidar>
-                <scan>
-                <horizontal>
-                    <samples>360</samples>
-                    <resolution>1.00000</resolution>
-                    <min_angle>0.000000</min_angle>
-                    <max_angle>6.280000</max_angle>
-                </horizontal>
-                </scan>
-                <range>
-                <min>0.120000</min>
-                <max>12.0</max>
-                <resolution>0.02</resolution>
-                </range>
-                <noise>
-                <type>gaussian</type>
-                <mean>0.0</mean>
-                <stddev>0.01</stddev>
-                </noise>
-            </lidar>
+            <update_rate>10.0</update_rate>
+            <topic>gps/data_raw</topic>
+            <navsat>
+                <position_sensing>
+                    <horizontal>
+                        <noise type="gaussian">
+                            <mean>0.0</mean>
+                            <stddev>0.00000027</stddev>
+                        </noise>
+                    </horizontal>
+                    <vertical>
+                        <noise type="gaussian">
+                            <mean>0.0</mean>
+                            <stddev>0.020</stddev>
+                        </noise>
+                    </vertical>
+                </position_sensing>
+            </navsat>
+            <gz_frame_id>gps_link</gz_frame_id>
         </sensor>
     </gazebo>
